Commit message: env_update

File: path_planner/robotv1.urdf (robot description, URDF)
Before this commit: robot rds_v1, 7 links, 6 joints
Joints:
- joint left_wheel_joint: limit (none) -> effort=100 velocity=100; type fixed -> continuous
- joint right_wheel_joint: limit (none) -> effort=100 velocity=100; type fixed -> continuous

Commit message: env updated v4

File: path_planner/robotv1.urdf (robot description, URDF)
Before this commit: robot rds_v1, 7 links, 6 joints
Links:
- link left_wheel: geometry collision cylinder length=0.05 radius=0.035; visual cylinder length=0.08 radius=0.035
- link right_wheel: geometry collision cylinder length=0.08 radius=0.035; visual cylinder length=0.1 radius=0.035
Joints:
- joint left_wheel_joint: axis (none) -> 0 0 1
- joint right_wheel_joint: axis (none) -> 0 0 1
